Commit message: adjust timing

File: ros/wc_ws/src/arm/my_robot/urdf/my_conveyor_belt.xacro (robot description, xacro)
@@ -6,6 +6,6 @@
     <xacro:property name="axle_length" value="0.03"/>
     <xacro:property name="axle_width" value="0.08"/>
-    <xacro:property name="axle_height" value="0.02"/>
-    <xacro:property name="arm_length" value="1.40"/>
+    <xacro:property name="axle_height" value="0.05"/>
+    <xacro:property name="arm_length" value="1.50"/>
     <xacro:property name="arm_width" value="0.032"/>
     <xacro:property name="arm_height" value="0.016"/>

File: ros/wc_ws/src/camera/yolobot_description/robot/yolobot.urdf (robot description, URDF)
Before this commit: robot yolobot, 4 links, 3 joints
Joints:
- joint rgb_cam_camera_link_joint: origin xyz=0.0 -3.0 1.55 rpy=0 0 0 -> xyz=0.0 -5.0 1.5 rpy=0 0 0
